File: DongleHiderPlus_PCB/DongleHiderPlus_PCB.kicad_pcb (KiCad board)
At the start: 4 copper layers, 28.2 x 26.1 mm, 23 parts, among them J1 USB3_A, J4 D-4, J5 D+4, P1 USB_C_Plug, U1 CH334F, U2 USBLC6-2SC6, Y1 12MHz

Commit message: add production files for rev 0.1
Routing:
- net GND: track 15.1 -> 16.7 mm
Other:
- board text added: "JLCJLCJLCJLC"
Changed lines of the file:
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@@
 		(layer "Edge.Cuts")
+	)
+	(gr_text "JLCJLCJLCJLC"
+		(at 101.579 76.1666 -0)
+		(layer "B.SilkS")
+		(effects
+			(font
+				(size 0.7 0.7)
+				(thickness 0.12)
+				(bold yes)
+			)
+			(justify bottom mirror)
+		)
 	)
 	(gr_text "V  - +  G"
@@
 	)
 	(segment
+		(start 108.0275 56.0783)
+		(end 106.8876 57.2182)
+		(width 0.5)
+		(layer "In1.Cu")
+		(net 1)
+	)
+	(segment
+		(start 108.0275 56.05)
+		(end 108.0275 56.0783)
+		(width 0.5)
+		(layer "In1.Cu")
+		(net 1)
+	)
+	(segment
 		(start 108.0275 56.05)
 		(end 108.0275 56.1291)
@@
 	)
 	(segment
+		(start 104.119 68.490505)
+		(end 104.884665 67.72484)
+		(width 0.127)
+		(layer "F.Cu")
+		(net 4)
+	)
+	(segment
+		(start 105.5312 73.6418)
+		(end 104.119 72.2296)
+		(width 0.127)
+		(layer "F.Cu")
+		(net 4)
+	)
+	(segment
+		(start 104.884665 67.72484)
+		(end 104.884665 64.342835)
+		(width 0.127)
+		(layer "F.Cu")
+		(net 4)
+	)
+	(segment
 		(start 104.884665 64.342835)
 		(end 105.9275 63.3)
@@
 	)
 	(segment
-		(start 103.992 72.1026)
-		(end 103.992 68.617505)
-		(width 0.127)
-		(layer "F.Cu")
-		(net 4)
-	)
-	(segment
-		(start 104.884665 67.72484)
-		(end 104.884665 64.342835)
+		(start 104.119 72.2296)
+		(end 104.119 68.490505)
 		(width 0.127)
 		(layer "F.Cu")
@@
 		(start 105.9275 63.3)
 		(end 106.5275 63.3)
-		(width 0.127)
-		(layer "F.Cu")
-		(net 4)
-	)
-	(segment
-		(start 103.992 68.617505)
-		(end 104.884665 67.72484)
-		(width 0.127)
-		(layer "F.Cu")
-		(net 4)
-	)
-	(segment
-		(start 105.5312 73.6418)
-		(end 103.992 72.1026)
 		(width 0.127)
 		(layer "F.Cu")
@@
 	)
 	(segment
+		(start 102.7372 73.6418)
+		(end 103.4387 73.6418)
+		(width 0.127)
+		(layer "F.Cu")
+		(net 32)
+	)
+	(segment
 		(start 96.4295 72.021)
-		(end 100.78981 72.021)
+		(end 101.1164 72.021)
 		(width 0.127)
 		(layer "F.Cu")
@@
 	)
 	(segment
-		(start 102.41061 73.6418)
-		(end 103.4387 73.6418)
+		(start 101.1164 72.021)
+		(end 102.7372 73.6418)
 		(width 0.127)
 		(layer "F.Cu")
@@
 	)
 	(segment
-		(start 100.78981 72.021)
-		(end 102.41061 73.6418)
-		(width 0.127)
-		(layer "F.Cu")
-		(net 32)
-	)
-	(segment
-		(start 100.9306 72.521)
-		(end 102.4426 74.033)
+		(start 102.4426 75.3284)
+		(end 102.656 75.5418)
+		(width 0.127)
+		(layer "F.Cu")
+		(net 33)
+	)
+	(segment
+		(start 101.0576 72.521)
+		(end 102.4426 73.906)
 		(width 0.127)
 		(layer "F.Cu")
@@
 	)
 	(segment
-		(start 102.4426 74.033)
+		(start 102.4426 73.906)
 		(end 102.4426 75.3284)
 		(width 0.127)
@@
 	(segment
 		(start 96.4295 72.521)
-		(end 100.9306 72.521)
-		(width 0.127)
-		(layer "F.Cu")
-		(net 33)
-	)
-	(segment
-		(start 102.4426 75.3284)
-		(end 102.656 75.5418)
-		(width 0.127)
-		(layer "F.Cu")
+		(end 101.0576 72.521)
+		(width 0.127)
+		(layer "F.Cu")
