File: DongleHiderPlus_PCB/DongleHiderPlus_PCB.kicad_pcb (KiCad board)
At the start: 4 copper layers, 28.2 x 26.1 mm, 23 parts, among them J1 USB3_A, J4 D-4, J5 D+4, P1 USB_C_Plug, U1 CH334F, U2 USBLC6-2SC6, Y1 12MHz

Commit message: add two empty middle layers to get JLC ENIG
Routing:
- added copper zone on In4.Cu, net GND
- removed copper zone on In2.Cu, net GND
Other:
- copper layers 4 -> 6
Changed lines of the file:
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@@
 		(1 "In1.Cu" signal)
 		(2 "In2.Cu" signal)
+		(3 "In3.Cu" signal)
+		(4 "In4.Cu" signal)
 		(31 "B.Cu" signal)
 		(32 "B.Adhes" user "B.Adhesive")
@@
 			(layer "dielectric 1"
 				(type "prepreg")
-				(thickness 0.2104)
+				(thickness 0.1)
 				(material "FR4")
 				(epsilon_r 4.5)
@@
 			(layer "dielectric 2"
 				(type "core")
-				(thickness 0.25)
+				(thickness 0.1504)
 				(material "FR4")
 				(epsilon_r 4.5)
@@
 			(layer "dielectric 3"
 				(type "prepreg")
-				(thickness 0.2104)
+				(thickness 0.1)
+				(material "FR4")
+				(epsilon_r 4.5)
+				(loss_tangent 0.02)
+			)
+			(layer "In3.Cu"
+				(type "copper")
+				(thickness 0.035)
+			)
+			(layer "dielectric 4"
+				(type "core")
+				(thickness 0.1504)
+				(material "FR4")
+				(epsilon_r 4.5)
+				(loss_tangent 0.02)
+			)
+			(layer "In4.Cu"
+				(type "copper")
+				(thickness 0.035)
+			)
+			(layer "dielectric 5"
+				(type "prepreg")
+				(thickness 0.1)
 				(material "FR4")
 				(epsilon_r 4.5)
@@
 			(size 2.2 2.2)
 			(drill 2.2)
-			(layers "*.Mask" "F.Cu" "In1.Cu" "In2.Cu" "B.Cu")
+			(layers "*.Mask" "F.Cu" "In1.Cu" "In4.Cu" "B.Cu")
 		)
 	)
@@
 		(end 108.0275 56.1291)
 		(width 0.5)
-		(layer "In2.Cu")
+		(layer "In4.Cu")
 		(net 1)
 	)
@@
 		(end 106.913 57.2436)
 		(width 0.5)
-		(layer "In2.Cu")
+		(layer "In4.Cu")
 		(net 1)
 	)
@@
 		(net 1)
 		(net_name "GND")
-		(layers "F.Cu" "In1.Cu" "In2.Cu" "B.Cu")
+		(layers "F.Cu" "In1.Cu" "In4.Cu" "B.Cu")
 		(name "GND")
 		(hatch edge 0.5)
